Commit message: adding world for training driving

File: description/robot_core.xacro (robot description, xacro)
@@ -11,4 +11,5 @@
             <origin xyz="0 0 0.0015" rpy="0 0 0" />
             <material name="gray" />
+        </visual>
         <collision>
             <geometry>
@@ -17,5 +18,4 @@
             <origin xyz="0 0 0.0015" rpy="0 0 0" />
         </collision>
-        </visual>
         <xacro:inertial_box mass=".09" x=".2" y=".24" z=".003">
             <origin xyz="0 0 0.0015" rpy="0 0 0"/>
