Commit message: created robot_core

File: description/robot.urdf.xacro (robot description, xacro)
@@ -1,4 +1,5 @@
 <?xml version="1.0"?>
 <robot xmlns:xacro="https://www.ros.org/wiki/xacro" name="robot">
-    <link name="base_link"/>
+    <!--this will be just the robot core components (excluding sensors and such)-->
+    <xacro:include filename="robot_core.xacro"/>
 </robot>

Commit message: gazebo simulation success

File: description/robot.urdf.xacro (robot description, xacro)
@@ -3,3 +3,4 @@
     <!--this will be just the robot core components (excluding sensors and such)-->
     <xacro:include filename="robot_core.xacro"/>
+    <xacro:include filename="gazebo_control.xacro"/>
 </robot>

File: description/robot_core.xacro (robot description, xacro)
@@ -3,7 +3,6 @@
     <xacro:include filename="robot_material.xacro"/>
     <xacro:include filename="inertial_macros.xacro"/>
-    <!-- My root link, being the footprint-->
-    <link name="base_footprint"/>
-    <link name="base_link">
+    <link name="base_link"/>
+    <link name="chassis_link">
         <visual>
             <geometry>
@@ -23,4 +22,12 @@
         </xacro:inertial_box>
     </link>
+    <joint name="chassis_joint" type="fixed">
+        <parent link="base_link"/>
+        <child link="chassis_link"/>
+        <origin xyz="0 0 0" rpy="0 0 0"/>
+    </joint>
+    <gazebo reference="base_link">
+        <material>Gazebo/White</material>
+    </gazebo>
     <link name="left_wheel_link">
         <visual>
@@ -28,5 +35,5 @@
                     <cylinder radius=".033" length="0.0254"/>
                 </geometry>
-                <origin xyz="0 0 0" rpy="-${pi/2} 0 0" />
+                <origin xyz="0 0 0" rpy="-0 0 0" />
                 <material name="black"/>
         </visual>
@@ -35,10 +42,20 @@
                 <cylinder radius=".033" length="0.0254"/>
             </geometry>
-            <origin xyz="0 0 0" rpy="-${pi/2} 0 0"/>
+            <origin xyz="0 0 0" rpy="0 0 0"/>
         </collision>
-        <xacro:inertial_cylinder mass=".0105" length=".0254" radius=".033">
-            <origin xyz="0 0 0 " rpy="-${pi/2} 0 0"/>
+        <xacro:inertial_cylinder mass=".1" length=".0254" radius=".033">
+            <origin xyz="0 0 0 " rpy="0 0 0"/>
         </xacro:inertial_cylinder>
     </link>
+    <joint name="base_left_wheel_joint" type="continuous">
+        <parent link="base_link"/>
+        <child link="left_wheel_link"/>
+        <origin xyz="0.06825 0.14143125 -.0145" rpy="-${pi/2} 0 0"/>
+        <axis xyz="0 0 1" />
+        <limit effort="30" velocity="10"/> <!--this will likely change, see urdf page. Effort could be set to estimated stall torque-->
+    </joint>
+    <gazebo reference="left_wheel_link">
+        <material>Gazebo/Black</material>
+    </gazebo>
     <link name="right_wheel_link">
         <visual>
@@ -46,5 +63,5 @@
                 <cylinder radius=".033" length="0.0254"/>
             </geometry>
-            <origin xyz="0 0 0" rpy="-${pi/2} 0 0" />
+            <origin xyz="0 0 0" rpy="0 0 0" />
             <material name="black"/>
         </visual>
@@ -53,10 +70,20 @@
                 <cylinder radius=".033" length="0.0254"/>
             </geometry>
-            <origin xyz="0 0 0" rpy="-${pi/2} 0 0"/>
+            <origin xyz="0 0 0" rpy="0 0 0"/>
         </collision>
-                <xacro:inertial_cylinder mass=".0105" length=".0254" radius=".033">
-            <origin xyz="0 0 0 " rpy="-${pi/2} 0 0"/>
+                <xacro:inertial_cylinder mass=".1" length=".0254" radius=".033">
+            <origin xyz="0 0 0 " rpy="0 0 0"/>
         </xacro:inertial_cylinder>
     </link>
+    <joint name="base_right_wheel_joint" type="continuous">
+        <parent link="base_link"/>
+        <child link="right_wheel_link"/>
+        <origin xyz="0.06825 -0.14143125 -.0145" rpy="${pi/2} 0 0"/>
+        <axis xyz="0 0 -1" />
+        <limit effort="30" velocity="10"/> <!--this will likely change, see urdf page. Effort could be set to estimated stall torque-->
+    </joint>
+    <gazebo reference="right_wheel_link">
+        <material>Gazebo/Black</material>
+    </gazebo>
     <link name="caster_wheel_link">
         <visual>
@@ -78,28 +105,8 @@
             <inertia ixx=".00000767125" ixy="0" ixz="0" iyy=".00000767125" iyz="0" izz=".00000767125"/>
         </inertial>
-        <xacro:inertial_sphere mass=".034" radius=".02375">
+        <xacro:inertial_sphere mass=".1" radius=".02375">
             <origin xyz="0 0 0" rpy="0 0 0"/>
         </xacro:inertial_sphere>
     </link>
-    <!-- original base joint -->
-    <joint name="base_joint" type="fixed">
-        <parent link="base_footprint"/>
-        <child link="base_link"/>
-        <origin xyz="0 0 .0475" rpy="0 0 0"/>
-    </joint>
-    <joint name="base_left_wheel_joint" type="continuous">
-        <parent link="base_link"/>
-        <child link="left_wheel_link"/>
-        <origin xyz="0.06825 0.14143125 -.0145" rpy="0 0 0"/>
-        <axis xyz="0 1 0" />
-        <limit effort="30" velocity="10"/> <!--this will likely change, see urdf page. Effort could be set to estimated stall torque-->
-    </joint>
-    <joint name="base_right_wheel_joint" type="continuous">
-        <parent link="base_link"/>
-        <child link="right_wheel_link"/>
-        <origin xyz="0.06825 -0.14143125 -.0145" rpy="0 0 0"/>
-        <axis xyz="0 1 0" />
-        <limit effort="30" velocity="10"/> <!--this will likely change, see urdf page. Effort could be set to estimated stall torque-->
-    </joint>
     <joint name="base_caster_wheel_joint" type="fixed">
         <parent link="base_link"/>
@@ -107,3 +114,6 @@
         <origin xyz="-0.0730125 0 -.02375" rpy="0 0 0"/>
     </joint>
+    <gazebo reference="caster_wheel_link">
+        <material>Gazebo/White</material>
+    </gazebo>
 </robot>

Commit message: ros2 control setup

File: description/robot.urdf.xacro (robot description, xacro)
@@ -3,4 +3,7 @@
     <!--this will be just the robot core components (excluding sensors and such)-->
     <xacro:include filename="robot_core.xacro"/>
-    <xacro:include filename="gazebo_control.xacro"/>
+    <!-- <xacro:include filename="gazebo_control.xacro"/> -->
+    <xacro:include filename="ros2_control.xacro" />
+    <!--now add another for the lidar sensor-->
+    <xacro:include filename="lidar.xacro"/>
 </robot>

File: description/robot_core.xacro (robot description, xacro)
@@ -35,5 +35,5 @@
                     <cylinder radius=".033" length="0.0254"/>
                 </geometry>
-                <origin xyz="0 0 0" rpy="-0 0 0" />
+                <origin xyz="0 0 0" rpy="0 0 0" />
                 <material name="black"/>
         </visual>

File: description/robot_material.xacro (robot description, xacro)
@@ -16,3 +16,6 @@
         <color rgba="0 0 0 1"/>
     </material>
+    <material name="red">
+        <color rgba="1 0 0 1"/>
+    </material>
 </robot>
